File: netzteil.sch (EAGLE design)
At the start: 49 parts, among them X1 NEB21R

Commit message: version v1 bestückt
Parts:
- C13: value 22n -> 5n
- R1: value 0,004 -> 0,005
- R10: value 5k1 -> 12k
- R11: value 73k2 -> 470k
- R12: value 8k06 -> 30k
- R16: value 51 -> 0
- R17: value 51 -> 330
- R18: value 8k06 -> 10k
- R2: value 0,009 -> 0,01
- R3: value 0,003 -> 0,004
- R5: value 866k -> 470k
- R6: value 1M -> 470k
- R7: value 576k -> 100k
- R8: value 57k6 -> 56k
Other:
- moved on the sheet: R18, SV2
Changed lines of the file:
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@@
 <part name="GND1" library="supply1" deviceset="GND" device=""/>
 <part name="GND3" library="supply1" deviceset="GND" device=""/>
-<part name="R1" library="resistor-shunt" deviceset="BVS" device="" value="0,004"/>
-<part name="R2" library="resistor-shunt" deviceset="BVS" device="" value="0,009"/>
-<part name="R3" library="resistor-shunt" deviceset="BVS" device="" value="0,003"/>
+<part name="R1" library="resistor-shunt" deviceset="BVS" device="" value="0,005"/>
+<part name="R2" library="resistor-shunt" deviceset="BVS" device="" value="0,01"/>
+<part name="R3" library="resistor-shunt" deviceset="BVS" device="" value="0,004"/>
 <part name="P+1" library="supply1" deviceset="+24V" device=""/>
 <part name="P+2" library="supply1" deviceset="+12V" device=""/>
@@
 <part name="C11" library="resistor" deviceset="C-EU" device="C0805K" value="100n"/>
 <part name="C12" library="resistor" deviceset="C-EU" device="C0805K" value="33n"/>
-<part name="C13" library="resistor" deviceset="C-EU" device="C0805K" value="22n"/>
+<part name="C13" library="resistor" deviceset="C-EU" device="C0805K" value="5n"/>
 <part name="R4" library="resistor" deviceset="R-EU_" device="M0805" value="51"/>
-<part name="R5" library="resistor" deviceset="R-EU_" device="M0805" value="866k"/>
-<part name="R6" library="resistor" deviceset="R-EU_" device="M0805" value="1M"/>
-<part name="R7" library="resistor" deviceset="R-EU_" device="M0805" value="576k"/>
-<part name="R8" library="resistor" deviceset="R-EU_" device="M0805" value="57k6"/>
+<part name="R5" library="resistor" deviceset="R-EU_" device="M0805" value="470k"/>
+<part name="R6" library="resistor" deviceset="R-EU_" device="M0805" value="470k"/>
+<part name="R7" library="resistor" deviceset="R-EU_" device="M0805" value="100k"/>
+<part name="R8" library="resistor" deviceset="R-EU_" device="M0805" value="56k"/>
 <part name="R9" library="resistor" deviceset="R-EU_" device="M0805" value="84k5"/>
-<part name="R10" library="resistor" deviceset="R-EU_" device="M0805" value="5k1"/>
-<part name="R11" library="resistor" deviceset="R-EU_" device="M0805" value="73k2"/>
-<part name="R12" library="resistor" deviceset="R-EU_" device="M0805" value="8k06"/>
+<part name="R10" library="resistor" deviceset="R-EU_" device="M0805" value="12k"/>
+<part name="R11" library="resistor" deviceset="R-EU_" device="M0805" value="470k"/>
+<part name="R12" library="resistor" deviceset="R-EU_" device="M0805" value="30k"/>
 <part name="R13" library="resistor" deviceset="R-EU_" device="M0805" value="200k"/>
 <part name="R14" library="resistor" deviceset="R-EU_" device="M0805" value="100k"/>
@@
 <part name="LED1" library="led" deviceset="LED" device="SML0805"/>
 <part name="LED2" library="led" deviceset="LED" device="SML0805"/>
-<part name="R16" library="resistor" deviceset="R-EU_" device="M0805" value="51"/>
-<part name="R17" library="resistor" deviceset="R-EU_" device="M0805" value="51"/>
+<part name="R16" library="resistor" deviceset="R-EU_" device="M0805" value="0"/>
+<part name="R17" library="resistor" deviceset="R-EU_" device="M0805" value="330"/>
 <part name="GND16" library="supply1" deviceset="GND" device=""/>
 <part name="P+3" library="supply1" deviceset="+5V" device=""/>
@@
 <part name="GND17" library="supply1" deviceset="GND" device=""/>
 <part name="P+11" library="supply1" deviceset="+24V" device=""/>
-<part name="R18" library="resistor" deviceset="R-EU_" device="M0805" value="8k06"/>
+<part name="R18" library="resistor" deviceset="R-EU_" device="M0805" value="10k"/>
 </parts>
 <sheets>
@@
 <instance part="P+9" gate="1" x="33.02" y="22.86"/>
 <instance part="P+10" gate="1" x="35.56" y="20.32"/>
-<instance part="SV2" gate="G$1" x="215.9" y="63.5" rot="R180"/>
+<instance part="SV2" gate="G$1" x="218.44" y="63.5" rot="R180"/>
 <instance part="LED1" gate="G$1" x="2.54" y="66.04"/>
 <instance part="LED2" gate="G$1" x="10.16" y="66.04"/>
@@
 <instance part="GND17" gate="1" x="17.78" y="111.76"/>
 <instance part="P+11" gate="1" x="25.4" y="111.76"/>
-<instance part="R18" gate="G$1" x="205.74" y="55.88" rot="R90"/>
+<instance part="R18" gate="G$1" x="208.28" y="55.88" rot="R90"/>
 </instances>
 <busses>
@@
 <pinref part="SV2" gate="G$1" pin="1"/>
 <wire x1="200.66" y1="78.74" x2="200.66" y2="76.2" width="0.1524" layer="91"/>
-<wire x1="208.28" y1="66.04" x2="205.74" y2="66.04" width="0.1524" layer="91"/>
+<wire x1="210.82" y1="66.04" x2="205.74" y2="66.04" width="0.1524" layer="91"/>
 <wire x1="205.74" y1="66.04" x2="205.74" y2="78.74" width="0.1524" layer="91"/>
 <wire x1="205.74" y1="78.74" x2="200.66" y2="78.74" width="0.1524" layer="91"/>
@@
 <pinref part="R12" gate="G$1" pin="1"/>
 <pinref part="GND14" gate="1" pin="GND"/>
-<wire x1="200.66" y1="50.8" x2="205.74" y2="50.8" width="0.1524" layer="91"/>
+<wire x1="200.66" y1="50.8" x2="208.28" y2="50.8" width="0.1524" layer="91"/>
 <junction x="200.66" y="50.8"/>
 <pinref part="R18" gate="G$1" pin="1"/>
@@
 <wire x1="195.58" y1="33.02" x2="104.14" y2="33.02" width="0.1524" layer="91"/>
 <pinref part="SV2" gate="G$1" pin="2"/>
-<wire x1="208.28" y1="63.5" x2="200.66" y2="63.5" width="0.1524" layer="91"/>
+<wire x1="210.82" y1="63.5" x2="200.66" y2="63.5" width="0.1524" layer="91"/>
 </segment>
 </net>
@@
 <segment>
 <pinref part="SV2" gate="G$1" pin="3"/>
-<wire x1="205.74" y1="60.96" x2="208.28" y2="60.96" width="0.1524" layer="91"/>
+<wire x1="208.28" y1="60.96" x2="210.82" y2="60.96" width="0.1524" layer="91"/>
 <pinref part="R18" gate="G$1" pin="2"/>
 </segment>

Commit message: version 2
Parts:
- removed U$2, U$3, U$6, U$7: STL100NH3LL, teile:STL100NH3LL
- removed U$4, U$5: SIA440DJ, teile:SIA440DJ
- added C17(OPT): 470n, resistor:C-EUC0805K
- added C18: 100µ, resistor:CPOL-EU153CLV-0605
- added C18(OPT): 100p, resistor:C-EUC0805K
- added D1, D2: (no value), diode:DIODE-SOD323-R
- added M1, M2, M3, M4: STL100NH3LL, teile:STL100NH3LL
- added R19: 4R7, resistor:R-EU_M0805
- added R20, R21(/OPT): 0, resistor:R-EU_M0805
- C16: value 100µ -> 470µ; device resistor:CPOL-EU153CLV-0807 -> resistor:CPOL-EU153CLV-1010
- D3, D4: value CGRM4001-G -> (none); device diode:CGRM4001-G -> diode:DIODE-SOD323-R
- R1, R2, R3: device resistor-shunt:BVS -> resistor:R-EU_R2512
- R16: value 0 -> 51
Connections:
- new net CLKOUT: U$1.CLKOUT
- new net GNDA: C11.2, C12.2, C18(OPT).2, LED1.C, R10.1, R12.1, R18.1, R21(/OPT).1, R7.1, R8.1, R9.1, SV1.1, U$1.SGND
- new net N$10: C17(OPT).1, R20.1, U$1.ISP
- new net N$9: C8.1, R19.1, U$1.VIN
- new net SYNC: R21(/OPT).2, U$1.SYNC
- net +12V: now also C17(OPT).2
- net BG1: now also M2.G; no longer U$5.G, U$7.G
- net BG2: now also M3.G; no longer U$3.G
- net GND: now also C18.-; no longer C11.2, C12.2, LED1.C, R10.1, R12.1, R18.1, R7.1, R8.1, R9.1, SV1.1, U$1.SGND, U$1.SYNC
- net ISP: now also D2.C, M4.D, R20.2; no longer U$1.ISP, U$2.D
- net N$8: now also C18(OPT).1
- net SNSP: now also D1.A, M2.S, M3.S; no longer U$3.S, U$5.S, U$7.S
- net SW1: now also D1.C, M1.S, M2.D; no longer U$4.S, U$5.D, U$6.S, U$7.D
- net SW2: now also D2.A, M3.D, M4.S; no longer U$2.S, U$3.D
- net TG1: now also M1.G; no longer U$4.G, U$6.G
- net TG2: now also M4.G; no longer U$2.G
- net VINN: now also C18.+, M1.D, R19.2; no longer C8.1, U$1.VIN, U$4.D, U$6.D
Other:
- note added: "(/OPT)"
- moved on the sheet: C12, C13, C9, R1, R10, R15, R2, R3, R4, R5, R6, R7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

Commit message: akkustecker
Parts:
- added U$2: MPX6P, con-ml:MPX6P
Connections:
- net +24V: now also U$2.1, U$2.2, U$2.3
- net GND: now also U$2.4, U$2.5, U$2.6
Changed lines of the file:
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@@
 <part name="GND9" library="supply1" deviceset="GNDA" device=""/>
 <part name="C18" library="resistor" deviceset="CPOL-EU" device="153CLV-0605" value="100µ"/>
+<part name="U$2" library="con-ml" deviceset="MPX6P" device=""/>
+<part name="GND18" library="supply1" deviceset="GND" device=""/>
+<part name="P+12" library="supply1" deviceset="+24V" device=""/>
 </parts>
 <sheets>
@@
 <instance part="GND9" gate="1" x="73.66" y="0"/>
 <instance part="C18" gate="G$1" x="127" y="111.76"/>
+<instance part="U$2" gate="G$1" x="162.56" y="12.7" rot="R180"/>
+<instance part="GND18" gate="1" x="162.56" y="-5.08"/>
+<instance part="P+12" gate="1" x="162.56" y="30.48"/>
 </instances>
 <busses>
@@
 <pinref part="P+11" gate="1" pin="+24V"/>
 <wire x1="30.48" y1="109.22" x2="25.4" y2="109.22" width="0.1524" layer="91"/>
+</segment>
+<segment>
+<pinref part="U$2" gate="G$1" pin="2"/>
+<wire x1="170.18" y1="15.24" x2="170.18" y2="25.4" width="0.1524" layer="91"/>
+<pinref part="P+12" gate="1" pin="+24V"/>
+<wire x1="170.18" y1="25.4" x2="162.56" y2="25.4" width="0.1524" layer="91"/>
+<wire x1="162.56" y1="25.4" x2="162.56" y2="27.94" width="0.1524" layer="91"/>
+<pinref part="U$2" gate="G$1" pin="1"/>
+<wire x1="162.56" y1="25.4" x2="162.56" y2="22.86" width="0.1524" layer="91"/>
+<junction x="162.56" y="25.4"/>
+<pinref part="U$2" gate="G$1" pin="3"/>
+<wire x1="162.56" y1="25.4" x2="154.94" y2="25.4" width="0.1524" layer="91"/>
+<wire x1="154.94" y1="25.4" x2="154.94" y2="15.24" width="0.1524" layer="91"/>
 </segment>
 </net>
@@
 <junction x="27.94" y="114.3"/>
 </segment>
-</net>
+<segment>
+<pinref part="U$2" gate="G$1" pin="4"/>
+<wire x1="170.18" y1="10.16" x2="170.18" y2="0" width="0.1524" layer="91"/>
+<pinref part="U$2" gate="G$1" pin="6"/>
+<wire x1="170.18" y1="0" x2="162.56" y2="0" width="0.1524" layer="91"/>
+<wire x1="162.56" y1="0" x2="162.56" y2="2.54" width="0.1524" layer="91"/>
+<pinref part="GND18" gate="1" pin="GND"/>
+<wire x1="162.56" y1="0" x2="162.56" y2="-2.54" width="0.1524" layer="91"/>
+<junction x="162.56" y="0"/>
+<pinref part="U$2" gate="G$1" pin="5"/>
+<wire x1="162.56" y1="0" x2="154.94" y2="0" width="0.1524" layer="91"/>
+<wire x1="154.94" y1="0" x2="154.94" y2="10.16" width="0.1524" layer="91"/>
+</segment>
+</net>

Commit message: enable/undervoltage on pin header
Parts:
- removed SV1: (no value), con-lstb:MA07-1
- added SV3: (no value), con-lstb:MA08-1
Connections:
- net +12V: now also SV3.3; no longer SV1.2
- net +24V: now also SV3.4; no longer SV1.3
- net +5V: now also SV3.5; no longer SV1.4
- net GNDA: now also SV3.2; no longer SV1.1
- net N$13: now also SV3.1
- net N$2: now also SV3.7; no longer SV1.6
- net N$25: now also SV3.6; no longer SV1.5
- net N$3: now also SV3.8; no longer SV1.7
Changed lines of the file:
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@@
 <part name="R15" library="resistor" deviceset="R-EU_" device="M0805" value="100k"/>
 <part name="C16" library="resistor" deviceset="CPOL-EU" device="153CLV-1010" value="470µ"/>
-<part name="SV1" library="con-lstb" deviceset="MA07-1" device=""/>
 <part name="P+8" library="supply1" deviceset="+5V" device=""/>
 <part name="P+9" library="supply1" deviceset="+24V" device=""/>
@@
 <part name="GND18" library="supply1" deviceset="GND" device=""/>
 <part name="P+12" library="supply1" deviceset="+24V" device=""/>
+<part name="SV3" library="con-lstb" deviceset="MA08-1" device=""/>
 </parts>
 <sheets>
@@
 <instance part="R15" gate="G$1" x="55.88" y="27.94" rot="R90"/>
 <instance part="C16" gate="G$1" x="200.66" y="109.22"/>
-<instance part="SV1" gate="1" x="12.7" y="22.86"/>
 <instance part="P+8" gate="1" x="30.48" y="25.4"/>
 <instance part="P+9" gate="1" x="33.02" y="22.86"/>
@@
 <instance part="GND18" gate="1" x="162.56" y="-5.08"/>
 <instance part="P+12" gate="1" x="162.56" y="30.48"/>
+<instance part="SV3" gate="1" x="12.7" y="20.32"/>
 </instances>
 <busses>
@@
 </segment>
 <segment>
-<pinref part="SV1" gate="1" pin="3"/>
 <pinref part="P+9" gate="1" pin="+24V"/>
 <wire x1="20.32" y1="20.32" x2="33.02" y2="20.32" width="0.1524" layer="91"/>
+<pinref part="SV3" gate="1" pin="4"/>
 </segment>
 <segment>
@@
 <segment>
 <pinref part="P+10" gate="1" pin="+12V"/>
-<pinref part="SV1" gate="1" pin="2"/>
 <wire x1="35.56" y1="17.78" x2="20.32" y2="17.78" width="0.1524" layer="91"/>
+<pinref part="SV3" gate="1" pin="3"/>
 </segment>
 </net>
@@
 <wire x1="63.5" y1="66.04" x2="17.78" y2="66.04" width="0.1524" layer="91"/>
 <junction x="17.78" y="66.04"/>
+<pinref part="SV3" gate="1" pin="1"/>
+<wire x1="20.32" y1="12.7" x2="20.32" y2="10.16" width="0.1524" layer="91"/>
+<wire x1="20.32" y1="10.16" x2="7.62" y2="10.16" width="0.1524" layer="91"/>
+<wire x1="7.62" y1="10.16" x2="7.62" y2="45.72" width="0.1524" layer="91"/>
+<wire x1="7.62" y1="45.72" x2="15.24" y2="45.72" width="0.1524" layer="91"/>
+<wire x1="15.24" y1="45.72" x2="15.24" y2="66.04" width="0.1524" layer="91"/>
+<wire x1="15.24" y1="66.04" x2="17.78" y2="66.04" width="0.1524" layer="91"/>
 </segment>
 </net>
@@
 <segment>
 <pinref part="P+8" gate="1" pin="+5V"/>
-<pinref part="SV1" gate="1" pin="4"/>
 <wire x1="30.48" y1="22.86" x2="20.32" y2="22.86" width="0.1524" layer="91"/>
+<pinref part="SV3" gate="1" pin="5"/>
 </segment>
 <segment>
@@
 <wire x1="40.64" y1="35.56" x2="38.1" y2="35.56" width="0.1524" layer="91"/>
 <wire x1="38.1" y1="35.56" x2="38.1" y2="25.4" width="0.1524" layer="91"/>
-<pinref part="SV1" gate="1" pin="5"/>
 <wire x1="38.1" y1="25.4" x2="20.32" y2="25.4" width="0.1524" layer="91"/>
 <wire x1="63.5" y1="38.1" x2="55.88" y2="38.1" width="0.1524" layer="91"/>
@@
 <wire x1="40.64" y1="40.64" x2="40.64" y2="35.56" width="0.1524" layer="91"/>
 <junction x="40.64" y="35.56"/>
+<pinref part="SV3" gate="1" pin="6"/>
 </segment>
 </net>
@@
 <pinref part="U$1" gate="G$1" pin="ISMON"/>
 <wire x1="35.56" y1="48.26" x2="63.5" y2="48.26" width="0.1524" layer="91"/>
-<pinref part="SV1" gate="1" pin="6"/>
 <wire x1="35.56" y1="27.94" x2="20.32" y2="27.94" width="0.1524" layer="91"/>
+<pinref part="SV3" gate="1" pin="7"/>
 </segment>
 </net>
@@
 <wire x1="63.5" y1="50.8" x2="33.02" y2="50.8" width="0.1524" layer="91"/>
 <wire x1="33.02" y1="50.8" x2="33.02" y2="30.48" width="0.1524" layer="91"/>
-<pinref part="SV1" gate="1" pin="7"/>
 <wire x1="33.02" y1="30.48" x2="20.32" y2="30.48" width="0.1524" layer="91"/>
+<pinref part="SV3" gate="1" pin="8"/>
 </segment>
 </net>
@@
 <net name="GNDA" class="0">
 <segment>
-<pinref part="SV1" gate="1" pin="1"/>
 <wire x1="20.32" y1="15.24" x2="22.86" y2="15.24" width="0.1524" layer="91"/>
 <pinref part="GND3" gate="1" pin="GNDA"/>
-</segment>
-<segment>
+<pinref part="SV3" gate="1" pin="2"/>
+</segment>
+<segment>
